Commit message: fix transform relation with rosbag

File: sim_ws/src/f1tenth_gym_ros/launch/ego_racecar.xacro (robot description, xacro)
@@ -27,10 +27,10 @@
     </visual>
   </link>
-  <joint name="base_to_laser_model" type="fixed">
+  <joint name="base_to_laser" type="fixed">
     <parent link="${car_name}/base_link"/>
-    <child link="${car_name}/laser_model"/>
+    <child link="${car_name}/laser"/>
     <origin xyz="${laser_distance_from_base_link} 0 ${ground_offset+height+(laser_height/2)}"/>
   </joint>
-  <link name="${car_name}/laser_model">
+  <link name="${car_name}/laser">
     <visual>
       <geometry>
